File: Electrical/Schematic/GenericWheatstoneBridge.sch (KiCad schematic (older format))
At the start: 38 parts

Commit message: Updates to Circuit Drawings
Update of circuit drawings and supporting files.  There will be at least
one more revision for final cleanup.
Parts:
- U? (x2): symbol ICS -> Ics
- U? (x2): symbol VS -> Vs
Changed lines of the file:
@@
 EESchema Schematic File Version 2
+LIBS:GenericWheatstoneBridge-rescue
 LIBS:power
 LIBS:device
@@
 LIBS:memory
 LIBS:xilinx
-LIBS:special
 LIBS:microcontrollers
 LIBS:dsp
@@
 LIBS:valves
 LIBS:NarwhalLib
-LIBS:noname-cache
-EELAYER 27 0
+LIBS:GenericWheatstoneBridge-cache
+EELAYER 25 0
 EELAYER END
-$Descr A4 11693 8268
+$Descr USLetter 11000 8500
 encoding utf-8
 Sheet 1 1
-Title "noname.sch"
-Date "20 sep 2015"
-Rev ""
+Title "Generic Wheatstone Bridge RTD Circuits"
+Date "2016-09-18"
+Rev "2"
 Comp ""
 Comment1 ""
@@
 Constant Current - 3 Wire RTD
 $Comp
-L ICS U?
+L Ics U?
 U 1 1 55FED564
 P 6400 5600
@@
 $EndComp
 $Comp
-L ICS U?
+L Ics U?
 U 1 1 55FEDC33
 P 2300 5550
@@
 $EndComp
 $Comp
-L VS U?
+L Vs U?
 U 1 1 55FEE2AE
 P 2300 2600
@@
 	3250 3500 3250 3350
 $Comp
-L VS U?
+L Vs U?
 U 1 1 55FEE7CB
 P 6400 2675
