File: Electrical/Schematic/FrontPanel.sch (KiCad schematic (older format))
At the start: 26 parts

Commit message: Final V1.0 Electrical Schematic and Parts List
Final version of electrical schematic and parts lists
Parts:
- removed P?: CONN_12X2, symbol CONN_12X2
- removed U? (x3): LTC4316F, ~, symbol LTC4316F
- added 22-01-2025, 22-23-2021: CONN_2, symbol CONN_2
- added 5103309-3: CONN_8X2, symbol CONN_8X2
- gave numbers to parts that had none: 6
Connections:
- wire segments 105 -> 87
Other:
- moved on the sheet: 22-01-2025, 22-23-2021

Commit message: Updated Schematic and Lots of New code
Parts:
- added 22-01-?, 22-23-?: CONN_2, symbol CONN_2
Connections:
- net +5V: now also 22-23-2021.1 (P1), 22-23-?.1 (P1)
- net at 5103309-3.6: now also 22-23-2021.2 (PM); no longer 22-23-2021.1 (P1)
- net at 5103309-3.8: now also 22-23-?.2 (PM); no longer 22-23-2021.2 (PM)
- net Pump Volt 1 renamed Pump Volt 1 (+)
- net Pump Volt 2 renamed Pump Volt 1 (-)
- new net Pump Volt 2 (+): 22-01-?.1 (P1)
- new net Pump Volt 2 (-): 22-01-?.2 (PM)
Changed lines of the file:
@@
 LIBS:atmel
 LIBS:valves
-LIBS:arduino_shieldsNCL
 LIBS:NarwhalLib
 LIBS:Project_Narwhal_Electrical-cache
@@
 Sheet 2 4
 Title "noname.sch"
-Date "11 oct 2015"
+Date "9 nov 2015"
 Rev ""
 Comp ""
@@
 $EndComp
 Text GLabel 8950 5350 2    50   Input ~ 0
-Pump Volt 1
+Pump Volt 1 (+)
 Text GLabel 8950 5550 2    50   Input ~ 0
-Pump Volt 2
+Pump Volt 1 (-)
 Text Notes 2950 1400 0    200  ~ 0
 Front Panel Connection Board
@@
 	8350 7250 1900 7250
 Wire Wire Line
-	4050 5350 7850 5350
-Wire Wire Line
-	4050 5450 7650 5450
-Wire Wire Line
-	7650 5450 7650 5550
-Wire Wire Line
-	7650 5550 7850 5550
-Wire Wire Line
 	7850 1750 4950 1750
 Wire Wire Line
@@
 Wire Wire Line
 	4500 5550 4050 5550
+$Comp
+L CONN_2 22-01-?
+U 1 1 56406421
+P 8500 5950
+F 0 "22-01-?" V 8450 5950 40  0000 C CNN
+F 1 "CONN_2" V 8550 5950 40  0000 C CNN
+F 2 "" H 8500 5950 60  0000 C CNN
+F 3 "" H 8500 5950 60  0000 C CNN
+	1    8500 5950
+	-1   0    0    -1
+$EndComp
+Text GLabel 8950 5850 2    50   Input ~ 0
+Pump Volt 2 (+)
+Text GLabel 8950 6050 2    50   Input ~ 0
+Pump Volt 2 (-)
+Wire Wire Line
+	8950 5850 8850 5850
+Wire Wire Line
+	8950 6050 8850 6050
+$Comp
+L CONN_2 22-23-?
+U 1 1 5640642B
+P 8200 5950
+F 0 "22-23-?" V 8150 5950 40  0000 C CNN
+F 1 "CONN_2" V 8250 5950 40  0000 C CNN
+F 2 "" H 8200 5950 60  0000 C CNN
+F 3 "" H 8200 5950 60  0000 C CNN
+	1    8200 5950
+	1    0    0    -1
+$EndComp
+Text GLabel 7750 5850 0    50   Input ~ 0
++5V
+Text GLabel 7750 5350 0    50   Input ~ 0
++5V
+Wire Wire Line
+	7850 5350 7750 5350
+Wire Wire Line
+	7750 5850 7850 5850
+Wire Wire Line
+	7250 5550 7850 5550
+Wire Wire Line
+	7150 6050 7850 6050
+Wire Wire Line
+	7250 5550 7250 5350
+Wire Wire Line
+	7250 5350 4050 5350
+Wire Wire Line
+	7150 6050 7150 5450
+Wire Wire Line
+	7150 5450 4050 5450
 $EndSCHEMATC

Commit message: Updates to Circuit Drawings
Update of circuit drawings and supporting files.  There will be at least
one more revision for final cleanup.
Parts:
- removed 22-01-2025, 22-01-?, 22-23-2021, 22-23-?: CONN_2, symbol CONN_2
- added K (x2): CONN_3, symbol CONN_3
- added U: RealTimeClock, symbol RealTimeClock
Connections:
- net +5V: now also K.1 (P1), U.~ (VCC)
- net ENC_A (BK): now also 22-23-2051.2
- net ENC_A (HLT): now also 22-23-2051.2
- net ENC_A (MLT): now also 22-23-2051.2
- net ENC_B (BK): now also 22-23-2051.3
- net ENC_B (HLT): now also 22-23-2051.3
- net ENC_B (MLT): now also 22-23-2051.3
- net ENC_GND (BK): now also 22-23-2051.1
- net ENC_GND (HLT): now also 22-23-2051.1
- net ENC_GND (MLT): now also 22-23-2051.1
- net ENC_SW1 (BK): now also 22-23-2051.4
- net ENC_SW1 (HLT): now also 22-23-2051.4
- net ENC_SW1 (MLT): now also 22-23-2051.4
- net ENC_SW2 (BK): now also 22-23-2051.5
- net ENC_SW2 (HLT): now also 22-23-2051.5
- net ENC_SW2 (MLT): now also 22-23-2051.5
- net Pump Volt 1 (-): now also K.2 (PM)
- net Pump Volt 2 (-): now also K.3 (P3)
- net ENC_GND (MAIN): now reaches 22-23-2051.1
- net ENC_A (MAIN): now reaches 22-23-2051.2
- net ENC_B (MAIN): now reaches 22-23-2051.3
- net ENC_SW1 (MAIN): now reaches 22-23-2051.4
- net ENC_SW2 (MAIN): now reaches 22-23-2051.5
- net at 22-23-2041.1 (P1), 22-23-2041.1 (P1), 22-23-2041.1 (P1)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: now also U.~ (VCC)
- net at 22-23-2041.2 (P2), 22-23-2041.2 (P2), 22-23-2041.2 (P2)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: now also U.~ (VCC)
- net at 5103309-3.6: now also K.2 (PM)
- net at 5103309-3.8: now also K.3 (P3)
- net GND renamed GND_5V
- net GND_5V: now also U.~ (VCC)
- new net Pump Volt (+): K.1 (P1)
Other:
- note added: "Note 1: Molex connector pin numbering convention: With female connector ears to the right, pin 1 is located at the top.\n Pin 1 is generally set as power."
- note added: "Note 2: GND_5V is the ground from the 5V step down voltage converter."
- note added: "Ribbon cable red\nstripe is Pin 1."
- moved on the sheet: 22-01-2025, 22-01-2045, 22-01-2055, 22-23-2021, 22-23-2041, 22-23-2051, 5103309-3

Commit message: Updated electrical drawings
Update to Arduino library
Updates power/grounds
Added pull down resistors to front panel
Added diff amp to main board
More clean up...
Parts:
- added R (x2): 2000, symbol R
Connections:
- net labels added: +5VLinear, GND_5VLinear
- net labels removed: +5V, GND_5V
- wire segments 99 -> 92
Other:
- moved on the sheet: 22-01-2025, 22-23-2021, 5103309-3
Changed lines of the file:
@@
 Sheet 2 4
 Title "Front Panel Connection Board"
-Date "2016-09-18"
-Rev "2"
+Date "2016-10-05"
+Rev "4"
 Comp "Project Narwhal"
 Comment1 ""
@@
 $EndComp
 Text GLabel 2500 4000 2    60   Input ~ 0
-GND_5V
+GND_5VLinear
 Text GLabel 2500 4600 2    60   Input ~ 0
-GND_5V
+GND_5VLinear
 Text GLabel 2500 4900 2    60   Input ~ 0
-GND_5V
+GND_5VLinear
 Text GLabel 2500 5200 2    60   Input ~ 0
-GND_5V
+GND_5VLinear
 Text GLabel 2500 5500 2    60   Input ~ 0
-GND_5V
+GND_5VLinear
 Text GLabel 2500 5750 2    60   Input ~ 0
-GND_5V
+GND_5VLinear
 Text GLabel 2500 6050 2    60   Input ~ 0
-GND_5V
+GND_5VLinear
 Text GLabel 2500 4300 2    60   Input ~ 0
-GND_5V
+GND_5VLinear
 Text GLabel 1350 4100 0    50   Input ~ 0
 ENC_A (HLT)
@@
 $EndComp
 Text GLabel 7750 1300 0    50   Input ~ 0
-+5V
++5VLinear
 Text GLabel 7750 1400 0    53   Input ~ 0
-GND_5V
+GND_5VLinear
 Text GLabel 9700 2700 2    50   Input ~ 0
 DISP_VCC (BK)
@@
 $EndComp
 Text GLabel 7750 2000 0    50   Input ~ 0
-+5V
++5VLinear
 Text GLabel 7750 2100 0    53   Input ~ 0
-GND_5V
+GND_5VLinear
 $Comp
 L CONN_4 22-23-2041
@@
 $EndComp
 Text GLabel 7750 2700 0    50   Input ~ 0
-+5V
++5VLinear
 Text GLabel 7750 2800 0    53   Input ~ 0
-GND_5V
+GND_5VLinear
 $Comp
 L CONN_4 22-23-2041
@@
 $EndComp
 Text GLabel 7750 3400 0    50   Input ~ 0
-+5V
++5VLinear
 Text GLabel 7750 3500 0    53   Input ~ 0
-GND_5V
+GND_5VLinear
 $Comp
 L CONN_2 22-01-2025
 U 1 1 561AFBF3
-P 1750 2700
-F 0 "22-01-2025" V 1700 2700 40  0000 C CNN
-F 1 "CONN_2" V 1800 2700 40  0000 C CNN
-F 2 "" H 1750 2700 60  0000 C CNN
-F 3 "" H 1750 2700 60  0000 C CNN
-	1    1750 2700
-	1    0    0    -1
-$EndComp
-Text GLabel 1300 2800 0    50   Input ~ 0
-GND_5V
-Text GLabel 1300 2600 0    50   Input ~ 0
-+5V
+P 8200 5700
+F 0 "22-01-2025" V 8150 5700 40  0000 C CNN
+F 1 "CONN_2" V 8250 5700 40  0000 C CNN
+F 2 "" H 8200 5700 60  0000 C CNN
+F 3 "" H 8200 5700 60  0000 C CNN
+	1    8200 5700
+	1    0    0    -1
+$EndComp
+Text GLabel 6450 5800 0    50   Input ~ 0
+GND_5VLinear
+Text GLabel 7750 5600 0    50   Input ~ 0
++5VLinear
 $Comp
 L CONN_2 22-23-2021
 U 1 1 561AFC02
-P 2050 2700
-F 0 "22-23-2021" V 2000 2700 40  0000 C CNN
-F 1 "CONN_2" V 2100 2700 40  0000 C CNN
-F 2 "" H 2050 2700 60  0000 C CNN
-F 3 "" H 2050 2700 60  0000 C CNN
-	1    2050 2700
+P 8500 5700
+F 0 "22-23-2021" V 8450 5700 40  0000 C CNN
+F 1 "CONN_2" V 8550 5700 40  0000 C CNN
+F 2 "" H 8500 5700 60  0000 C CNN
+F 3 "" H 8500 5700 60  0000 C CNN
+	1    8500 5700
 	-1   0    0    -1
 $EndComp
-Text GLabel 2500 2600 2    50   Input ~ 0
-+5V
-Text GLabel 2500 2800 2    50   Input ~ 0
-GND_5V
+Text GLabel 8950 5600 2    50   Input ~ 0
++5VLinear
+Text GLabel 8950 5800 2    50   Input ~ 0
+GND_5VLinear
 $Comp
 L CONN_8X2 5103309-3
 U 1 1 561AFC12
-P 3650 4850
-F 0 "5103309-3" H 3650 5300 60  0000 C CNN
-F 1 "CONN_8X2" V 3650 4850 50  0000 C CNN
-F 2 "" H 3650 4850 60  0000 C CNN
-F 3 "" H 3650 4850 60  0000 C CNN
-	1    3650 4850
+P 4250 4850
+F 0 "5103309-3" H 4250 5300 60  0000 C CNN
+F 1 "CONN_8X2" V 4250 4850 50  0000 C CNN
+F 2 "" H 4250 4850 60  0000 C CNN
+F 3 "" H 4250 4850 60  0000 C CNN
+	1    4250 4850
 	1    0    0    -1
 $EndComp
@@
 	8350 6600 1900 6600
 Wire Wire Line
-	4200 1100 4950 1100
-Wire Wire Line
-	4950 1100 7850 1100
-Wire Wire Line
-	4950 1100 4950 1800
-Wire Wire Line
-	4950 1800 4950 2500
-Wire Wire Line
-	4950 2500 4950 3200
-Wire Wire Line
-	4950 3200 4950 4500
-Wire Wire Line
-	4950 4500 4050 4500
-Wire Wire Line
-	5050 4600 4050 4600
-Wire Wire Line
-	5050 1200 5050 1900
-Wire Wire Line
-	5050 1900 5050 2600
-Wire Wire Line
-	5050 2600 5050 3300
-Wire Wire Line
-	5050 3300 5050 4600
-Wire Wire Line
-	4200 1200 5050 1200
-Wire Wire Line
-	5050 1200 7850 1200
+	4200 1100 7850 1100
+Wire Wire Line
+	4950 1100 4950 4500
+Wire Wire Line
+	4950 4500 4650 4500
+Wire Wire Line
+	5050 4600 4650 4600
+Wire Wire Line
+	5050 1200 5050 4600
+Wire Wire Line
+	4200 1200 7850 1200
 Wire Wire Line
 	7850 1800 4950 1800
@@
 Connection ~ 5050 3300
 Wire Wire Line
-	1300 2800 1400 2800
-Wire Wire Line
-	1300 2600 1400 2600
-Wire Wire Line
-	2500 2600 2400 2600
-Wire Wire Line
-	2500 2800 2400 2800
-Wire Wire Line
-	3250 4500 3250 4100
-Wire Wire Line
-	3250 4100 2450 4100
-Wire Wire Line
-	3250 4600 3200 4600
-Wire Wire Line
-	3200 4600 3200 4200
-Wire Wire Line
-	3200 4200 2450 4200
-Wire Wire Line
-	3250 4700 3150 4700
-Wire Wire Line
-	3150 4700 3150 4400
-Wire Wire Line
-	3150 4400 2450 4400
-Wire Wire Line
-	3250 4800 3100 4800
-Wire Wire Line
-	3100 4800 3100 4700
-Wire Wire Line
-	3100 4700 2450 4700
-Wire Wire Line
-	3250 4900 3050 4900
-Wire Wire Line
-	3050 4900 3050 4800
-Wire Wire Line
-	3050 4800 2450 4800
-Wire Wire Line
-	3250 5000 2450 5000
-Wire Wire Line
-	2450 5300 3050 5300
-Wire Wire Line
-	3050 5300 3050 5100
-Wire Wire Line
-	3050 5100 3250 5100
-Wire Wire Line
-	2450 5400 3100 5400
-Wire Wire Line
-	3100 5400 3100 5200
-Wire Wire Line
-	3100 5200 3250 5200
-Wire Wire Line
-	2450 5600 4200 5600
-Wire Wire Line
-	4200 5600 4200 5200
-Wire Wire Line
-	4200 5200 4050 5200
-Wire Wire Line
-	2450 5850 4300 5850
-Wire Wire Line
-	4300 5850 4300 5100
-Wire Wire Line
-	4300 5100 4050 5100
-Wire Wire Line
-	2450 5950 4400 5950
-Wire Wire Line
-	4400 5950 4400 5000
-Wire Wire Line
-	4400 5000 4050 5000
-Wire Wire Line
-	2450 6150 4500 6150
-Wire Wire Line
-	4500 6150 4500 4900
-Wire Wire Line
-	4500 4900 4050 4900
+	6450 5800 7850 5800
+Wire Wire Line
+	7750 5600 7850 5600
+Wire Wire Line
+	8950 5600 8850 5600
+Wire Wire Line
+	8950 5800 8850 5800
+Wire Wire Line
+	3750 4500 3750 4100
+Wire Wire Line
+	3750 4100 2450 4100
+Wire Wire Line
+	3850 4600 3700 4600
+Wire Wire Line
+	3700 4600 3700 4200
+Wire Wire Line
+	3700 4200 2450 4200
+Wire Wire Line
+	3850 4700 3650 4700
+Wire Wire Line
+	3650 4700 3650 4400
+Wire Wire Line
+	3650 4400 2450 4400
+Wire Wire Line
+	3850 4800 3600 4800
+Wire Wire Line
+	3600 4800 3600 4700
+Wire Wire Line
+	3600 4700 2450 4700
+Wire Wire Line
+	3850 4900 3550 4900
+Wire Wire Line
+	3550 4900 3550 4800
+Wire Wire Line
+	3550 4800 2450 4800
+Wire Wire Line
+	3850 5000 2450 5000
+Wire Wire Line
+	2450 5300 3650 5300
+Wire Wire Line
+	3650 5300 3650 5100
+Wire Wire Line
+	3650 5100 3850 5100
+Wire Wire Line
+	2450 5400 3750 5400
+Wire Wire Line
+	3750 5400 3750 5200
+Wire Wire Line
+	3750 5200 3850 5200
+Wire Wire Line
+	2450 5600 4750 5600
+Wire Wire Line
+	4750 5600 4750 5200
+Wire Wire Line
+	4750 5200 4650 5200
+Wire Wire Line
+	2450 5850 4850 5850
+Wire Wire Line
+	4850 5850 4850 5100
+Wire Wire Line
+	4850 5100 4650 5100
+Wire Wire Line
+	2450 5950 4950 5950
+Wire Wire Line
+	4950 5950 4950 5000
+Wire Wire Line
+	4950 5000 4650 5000
+Wire Wire Line
+	2450 6150 5050 6150
+Wire Wire Line
+	5050 6150 5050 4900
+Wire Wire Line
+	5050 4900 4650 4900
 Text GLabel 8950 4800 2    50   Input ~ 0
 Pump Volt 2 (-)
 Text GLabel 7750 4600 0    50   Input ~ 0
-+5V
-Wire Wire Line
-	7250 4700 7850 4700
-Wire Wire Line
-	7150 4800 7850 4800
-Wire Wire Line
-	7250 4700 7250 4700
-Wire Wire Line
-	7250 4700 4050 4700
-Wire Wire Line
-	7150 4800 7150 4800
-Wire Wire Line
-	7150 4800 4050 4800
++5VLinear
+Wire Wire Line
+	4650 4700 7850 4700
+Wire Wire Line
+	4650 4800 7850 4800
 Text Notes 600  7600 0    60   ~ 0
 Note 1: Molex connector pin numbering convention: With female connector ears to the right, pin 1 is located at the top.\n        Pin 1 is generally set as power.
@@
 Note 2: GND_5V is the ground from the 5V step down voltage converter.
 Text GLabel 4200 1400 2    50   Input ~ 0
-GND_5V
+GND_5VLinear
 Text GLabel 4200 1300 2    50   Input ~ 0
-+5V
++5VLinear
 Connection ~ 4950 1100
 Connection ~ 5050 1200
-Text Notes 3400 4300 0    60   ~ 0
+Text Notes 3950 4250 0    60   ~ 0
 Ribbon cable red\nstripe is Pin 1.
 $Comp
@@
 Wire Wire Line
 	8850 4800 8950 4800
+$Comp
+L R R
+U 1 1 57F1B0D5
+P 6700 5150
+F 0 "R" V 6780 5150 50  0000 C CNN
+F 1 "2000" V 6700 5150 50  0000 C CNN
+F 2 "" V 6630 5150 50  0000 C CNN
+F 3 "" H 6700 5150 50  0000 C CNN
+	1    6700 5150
+	1    0    0    -1
+$EndComp
+$Comp
+L R R
+U 1 1 57F1B148
+P 6900 5400
+F 0 "R" V 6980 5400 50  0000 C CNN
+F 1 "2000" V 6900 5400 50  0000 C CNN
+F 2 "" V 6830 5400 50  0000 C CNN
+F 3 "" H 6900 5400 50  0000 C CNN
+	1    6900 5400
+	1    0    0    -1
+$EndComp
+Wire Wire Line
+	6700 5000 6700 4700
+Connection ~ 6700 4700
+Wire Wire Line
+	6700 5300 6700 5800
+Connection ~ 6700 5800
+Wire Wire Line
+	6900 4800 6900 5250
+Connection ~ 6900 4800
+Wire Wire Line
+	6900 5550 6900 5800
+Connection ~ 6900 5800
+Wire Wire Line
+	3750 4500 3850 4500
 $EndSCHEMATC

Commit message: Updated schematics and documentation
Updated schematics and documentation
Parts:
- R: value 2000 -> 1800
Changed lines of the file:
@@
 Sheet 2 4
 Title "Front Panel Connection Board"
-Date "2016-10-05"
-Rev "4"
+Date "2016-10-30"
+Rev "5"
 Comp "Project Narwhal"
 Comment1 ""
@@
 P 6700 5150
 F 0 "R" V 6780 5150 50  0000 C CNN
-F 1 "2000" V 6700 5150 50  0000 C CNN
+F 1 "1800" V 6700 5150 50  0000 C CNN
 F 2 "" V 6630 5150 50  0000 C CNN
 F 3 "" H 6700 5150 50  0000 C CNN
@@
 P 6900 5400
 F 0 "R" V 6980 5400 50  0000 C CNN
-F 1 "2000" V 6900 5400 50  0000 C CNN
+F 1 "1800" V 6900 5400 50  0000 C CNN
 F 2 "" V 6830 5400 50  0000 C CNN
 F 3 "" H 6900 5400 50  0000 C CNN
