File: Electrical/Schematic/Project_Narwhal_Electrical.sch (KiCad schematic (older format))
At the start: 41 parts

Commit message: Final V1.0 Electrical Schematic and Parts List
Final version of electrical schematic and parts lists
Parts:
- removed P? (x2): CONN_2, symbol CONN_2
- removed P?: CONN_12X2, symbol CONN_12X2
- removed P? (x6): CONN_5, symbol CONN_5
- added 22-01-2075 (x4), 22-23-2071 (x2): CONN_7, symbol CONN_7
- added 5103309-3: CONN_8X2, symbol CONN_8X2
- gave numbers to parts that had none: 6
Connections:
- net labels removed: BK I2C Trans EN, I2C Trans 1 Enable, I2C Trans 2 Enable, I2C Trans 3 Enable, MLT I2C Trans EN, TIMER I2C Trans EN
- wire segments 252 -> 245
Other:
- moved on the sheet: 22-01-2035, 22-01-2105, Onboard

Commit message: Updated Schematic and Lots of New code
Parts:
- removed R? (x3): R, ~, symbol R
- removed U? (x3): AD623, symbol AD623
- added U? (x2): CONN_2, symbol CONN_2
- added U?: SDCARD, symbol SDCARD
Connections:
- net labels added: +3.3V
- net labels removed: RB1_EN0, RB1_EN1, RB1_EN2, RB1_EN3, RB1_EN4, RB1_EN5, RB1_EN6, RB1_EN7, RB2_EN0, RB2_EN1, RB2_EN2, RB2_EN3, RB2_EN4, RB2_EN5, RB2_EN6, RB2_EN7
- wire segments 245 -> 230
Other:
- moved on the sheet: 22-01-2025, 22-23-2021

Commit message: Updates to Circuit Drawings
Update of circuit drawings and supporting files.  There will be at least
one more revision for final cleanup.
Parts:
- added 12V: PowerSupply, symbol PowerSupply
- added P (x2): CONN_2, symbol CONN_2
- gave numbers to parts that had none: 2
Connections:
- net labels added: Alarm1, Alarm2, BK_PilotLight, BK_Sol1, BK_Sol2, GND_12V, GND_5V, GND_??V, HLT_PilotLight, HLT_Sol1, HLT_Sol2, MLT_PilotLight, MLT_Sol1, MLT_Sol2, PL1_AN_(HLT_TC), PL2_AN_(MLT_TC), PL3_AN_(BK_TC), Spare
- net labels removed: EN0 (RB2), EN1 (RB2), EN2 (RB1), EN2 (RB2), EN3 (RB1), EN3 (RB2), EN4 (RB1), EN4 (RB2), EN5 (RB1), EN5 (RB2), EN6 (RB1), EN6 (RB2), EN7 (RB1), EN7 (RB2), GND, GND (RB1), GND (RB2), PL1_AN, PL2_AN, PL3_AN, VCC (RB2)
- wire segments 230 -> 220
Other:
- note added: "Arduino Mega Shield"
- note added: "Blue"
- note added: "C"
- note added: "G"
- note added: "L"
- note added: "Note 1: Molex connector pin numbering convention: With female connector ears to the right, pin 1 is located at the top.\n Pin 1 is generally set as power."
- note added: "Note 2: GND_12V is the ground from the 12V power supply. GND_5V is the ground from the 5V step down voltage converter."
- note added: "Quick Disconnect\nPin Out"
- note added: "R"
- note added: "Ribbon cable red\nstripe is Pin 1."
- note added: "S"
- note added: "T"
- note added: "Yellow"
- note removed: "Narwhal Arduino Mega Shield"
- moved on the sheet: 22-01-2025, 22-23-2021, U

Commit message: Updated electrical drawings
Update to Arduino library
Updates power/grounds
Added pull down resistors to front panel
Added diff amp to main board
More clean up...
Parts:
- removed 22-01-2025 (x4), 22-23-2021 (x3), U: CONN_2, symbol CONN_2
- added 22-01 (x6), 22-23-?, U?: CONN_2, symbol CONN_2
- added C (x3): 0.1uF, symbol C
- added R (x9): 2000, symbol R
- added U? (x3): AD623, symbol AD623
- renumbered 12V to 12V~Linear~Power~Supply
Connections:
- net labels added: +12VLinear, +3.3VArduino, +5VArduino, +5VLinear, CS, GND_120VAC, GND_12VLinear, GND_5VLinear, MISO, MOSI, PilotLight_1_AN_(HLT_TC), PilotLight_2_AN_(MLT_TC), PilotLight_3_AN_(BK_TC), SCK
- net labels removed: +12V, +3.3V, +5V, GND_12V, GND_5V, GND_??V, PL1_AN_(HLT_TC), PL2_AN_(MLT_TC), PL3_AN_(BK_TC)
- wire segments 220 -> 280
Other:
- note added: "SD Card\nConnections"
- moved on the sheet: 12V Linear Power Supply, 22-01-2035, 22-01-2075, 22-01-2105, 22-23-2021, 22-23-2071, 22-23-2101, 5103309-3, Onboard, P, SHIELD, U

Commit message: Updated schematics and documentation
Updated schematics and documentation
Parts:
- renumbered 12V~Linear~Power~Supply to 12V
Connections:
- wire segments 280 -> 285
Other:
- moved on the sheet: 12V
Changed lines of the file:
@@
 Sheet 1 4
 Title "Arduino Mega Shield"
-Date "2016-10-05"
-Rev "3"
+Date "2016-10-30"
+Rev "4"
 Comp "Project Narwhal"
 Comment1 ""
@@
 L EA50-5V U?
 U 1 1 55E66878
-P 8750 9800
-F 0 "U?" H 8750 9800 60  0001 C CNN
-F 1 "EA50-5V" H 8750 9800 60  0000 C CNN
-F 2 "" H 8750 9800 60  0000 C CNN
-F 3 "" H 8750 9800 60  0000 C CNN
-	1    8750 9800
-	-1   0    0    -1
-$EndComp
-Text GLabel 8150 9600 0    60   Input ~ 0
+P 10250 9800
+F 0 "U?" H 10250 9800 60  0001 C CNN
+F 1 "EA50-5V" H 10250 9800 60  0000 C CNN
+F 2 "" H 10250 9800 60  0000 C CNN
+F 3 "" H 10250 9800 60  0000 C CNN
+	1    10250 9800
+	1    0    0    -1
+$EndComp
+Text GLabel 10850 9600 2    60   Input ~ 0
 +5VLinear
-Text GLabel 8150 10000 0    60   Input ~ 0
+Text GLabel 10850 10000 2    60   Input ~ 0
 GND_5VLinear
 Text GLabel 2550 7000 0    47   Input ~ 0
@@
 GND_5VLinear
 $Comp
-L PowerSupply 12V~Linear~Power~Supply
+L PowerSupply 12V
 U 1 1 57E3A5DF
-P 10850 9800
-F 0 "12V Linear Power Supply" H 10850 9600 60  0000 C CNN
-F 1 "PowerSupply" H 10850 10000 60  0000 C CNN
-F 2 "" H 10850 9800 60  0000 C CNN
-F 3 "" H 10850 9800 60  0000 C CNN
-	1    10850 9800
-	1    0    0    -1
-$EndComp
-Text GLabel 9950 9700 0    60   Input ~ 0
+P 8150 9800
+F 0 "12V" H 8150 9600 60  0000 C CNN
+F 1 "PowerSupply" H 8150 10000 60  0000 C CNN
+F 2 "" H 8150 9800 60  0000 C CNN
+F 3 "" H 8150 9800 60  0000 C CNN
+	1    8150 9800
+	-1   0    0    -1
+$EndComp
+Text GLabel 9200 9350 2    60   Input ~ 0
 +12VLinear
-Text GLabel 9950 9900 0    60   Input ~ 0
+Text GLabel 9200 10250 2    60   Input ~ 0
 GND_12VLinear
 Wire Wire Line
@@
 Wire Wire Line
 	10450 2400 10600 2400
-Wire Wire Line
-	9350 9600 10050 9600
-Wire Wire Line
-	10050 10000 9350 10000
-Wire Wire Line
-	10050 9600 10050 9750
-Connection ~ 10050 9700
-Wire Wire Line
-	10050 9850 10050 10000
-Connection ~ 10050 9900
-Wire Wire Line
-	9950 9700 10050 9700
-Wire Wire Line
-	9950 9900 10050 9900
 Text GLabel 5650 7700 2    60   Input ~ 0
 GND_5VLinear
@@
 	6650 4350 6650 4200
 Connection ~ 8250 4350
-Text GLabel 6250 4000 0    60   Input ~ 0
-GND_120VAC
-Wire Wire Line
-	6250 4000 6300 4000
+Wire Wire Line
+	5700 4000 6300 4000
 Wire Wire Line
 	6600 4000 6650 4000
@@
 	-1   0    0    -1
 $EndComp
-Text GLabel 5700 6150 2    60   Input ~ 0
+Text GLabel 5900 6150 2    60   Input ~ 0
 GND_120VAC
 Text GLabel 14250 2450 2    60   Input ~ 0
@@
 	6650 5300 6650 5150
 Connection ~ 8250 5300
-Text GLabel 6250 4950 0    60   Input ~ 0
-GND_120VAC
-Wire Wire Line
-	6250 4950 6300 4950
+Wire Wire Line
+	5700 4950 6300 4950
 Wire Wire Line
 	6600 4950 6650 4950
@@
 	6650 6200 6650 6050
 Connection ~ 8250 6200
-Text GLabel 6250 5850 0    60   Input ~ 0
+Wire Wire Line
+	5700 5850 6300 5850
+Wire Wire Line
+	6600 5850 6650 5850
+Wire Wire Line
+	6600 5950 6650 5950
+Text GLabel 5900 4300 2    60   Input ~ 0
 GND_120VAC
-Wire Wire Line
-	6250 5850 6300 5850
-Wire Wire Line
-	6600 5850 6650 5850
-Wire Wire Line
-	6600 5950 6650 5950
-Text GLabel 5700 4300 2    60   Input ~ 0
-GND_120VAC
-Text GLabel 5700 5250 2    60   Input ~ 0
+Text GLabel 5900 5250 2    60   Input ~ 0
 GND_120VAC
 Text Notes 4200 5500 0    60   ~ 0
@@
 	5600 4100 6300 4100
 Wire Wire Line
-	5600 4300 5700 4300
+	5600 4300 5900 4300
 Wire Wire Line
 	5600 5050 6300 5050
 Wire Wire Line
-	5600 5250 5700 5250
+	5600 5250 5900 5250
 Wire Wire Line
 	5600 5950 6300 5950
 Wire Wire Line
-	5600 6150 5700 6150
+	5600 6150 5900 6150
 Wire Wire Line
 	9300 5950 8200 5950
@@
 Text Notes 9650 5100 0    60   ~ 0
 SD Card\nConnections
+Text GLabel 8800 10250 0    60   Input ~ 0
+GND_120VAC
+Wire Wire Line
+	9100 9750 8950 9750
+Wire Wire Line
+	9100 9350 9100 9750
+Wire Wire Line
+	9100 9600 9650 9600
+Wire Wire Line
+	8950 9850 9100 9850
+Wire Wire Line
+	9100 9850 9100 10250
+Wire Wire Line
+	9100 9350 9200 9350
+Connection ~ 9100 9600
+Wire Wire Line
+	8800 10250 9200 10250
+Connection ~ 9100 10000
+Wire Wire Line
+	9100 10000 9650 10000
+Connection ~ 9100 10250
+Wire Wire Line
+	5700 4300 5700 4000
+Connection ~ 5700 4300
+Wire Wire Line
+	5700 5250 5700 4950
+Connection ~ 5700 5250
+Wire Wire Line
+	5700 6150 5700 5850
+Connection ~ 5700 6150
 $EndSCHEMATC
