File: Electrical/Schematic/RTDSenseCircuit.sch (KiCad schematic (older format))
At the start: 27 parts

Commit message: Final V1.0 Electrical Schematic and Parts List
Final version of electrical schematic and parts lists
Parts:
- removed P?: CONN_2, symbol CONN_2
- removed P?: CONN_5, symbol CONN_5
- added 22-23-2071: CONN_7, symbol CONN_7
- added R? (x4): 5, ~, symbol R
- R? (x4): value R -> 100
- R? (x8): value R -> 2000
- R? (x4): value R -> 2500
- gave numbers to parts that had none: 1
Connections:
- net labels added: Vs
- net labels removed: RTD0_C, RTD1_C, RTD2_C, RTD3_C, Vin
- wire segments 140 -> 145
Other:
- moved on the sheet: 22-23-2031

Commit message: Updated Schematic and Lots of New code
Parts:
- added C, C? (x3): 0.1uF, ~, symbol C
- R? (x4): value 2500 -> 2000
Connections:
- wire segments 145 -> 149
Other:
- moved on the sheet: 22-23-2031

Commit message: Updates to Circuit Drawings
Update of circuit drawings and supporting files.  There will be at least
one more revision for final cleanup.
Parts:
- added C: 10uF, ~, symbol C-RESCUE-Project_Narwhal_Electrical
- added R (x8): 2000, ~, symbol R-RESCUE-Project_Narwhal_Electrical
- C: symbol C -> C-RESCUE-Project_Narwhal_Electrical
- C: renamed from C?; symbol C -> C-RESCUE-Project_Narwhal_Electrical
- R, R2, R3, R4: renamed from R?; symbol R -> R-RESCUE-Project_Narwhal_Electrical
Connections:
- net labels added: +12V, GND_12V
- net labels removed: GND, Vs
- wire segments 149 -> 189
Other:
- note added: "Note 1: Molex connector pin numbering convention: With female connector ears to the right, pin 1 is located at the top.\n Pin 1 is generally set as power."
- note added: "Note 2: GND_12V is the ground from the 12V power supply."
- note added: "Note 3: Molex #1 connector is #2 on RTD cable (white wire)."
- note added: "Note 4: 5 Ohm resistor added such that zero deg C equals a positive voltage allowing for calibration in the software\n (Arduino cannot read negative voltage)"
- moved on the sheet: P

Commit message: Updated electrical drawings
Update to Arduino library
Updates power/grounds
Added pull down resistors to front panel
Added diff amp to main board
More clean up...
Changed lines of the file:
@@
 	2050 2600 2700 2600
 Wire Wire Line
-	3200 2600 3450 2600
-Wire Wire Line
-	3450 2600 3550 2600
+	3200 2600 3550 2600
 Wire Wire Line
 	4750 2750 4500 2750
 Wire Wire Line
-	4750 2600 4750 2650
-Wire Wire Line
-	4750 2650 4750 2750
+	4750 2600 4750 2750
 Wire Wire Line
 	4750 2600 4600 2600
@@
 	2050 3750 2700 3750
 Wire Wire Line
-	3200 3750 3450 3750
-Wire Wire Line
-	3450 3750 3550 3750
+	3200 3750 3550 3750
 Wire Wire Line
 	4600 3750 4750 3750
 Wire Wire Line
-	4750 3750 4750 3800
-Wire Wire Line
-	4750 3800 4750 3900
+	4750 3750 4750 3900
 Wire Wire Line
 	2050 4850 2700 4850
 Wire Wire Line
-	3200 4850 3450 4850
-Wire Wire Line
-	3450 4850 3550 4850
+	3200 4850 3550 4850
 Wire Wire Line
 	4600 4850 4750 4850
 Wire Wire Line
-	4750 4850 4750 4900
-Wire Wire Line
-	4750 4900 4750 5000
+	4750 4850 4750 5000
 Wire Wire Line
 	4800 3800 4750 3800
@@
 	2050 5900 2700 5900
 Wire Wire Line
-	3200 5900 3450 5900
-Wire Wire Line
-	3450 5900 3550 5900
+	3200 5900 3550 5900
 Wire Wire Line
 	4600 5900 4750 5900
 Wire Wire Line
-	4750 5900 4750 5950
-Wire Wire Line
-	4750 5950 4750 6050
+	4750 5900 4750 6050
 Wire Wire Line
 	4800 5950 4750 5950
@@
 	7250 4950 8400 4950
 Wire Wire Line
-	7250 4850 7650 4850
-Wire Wire Line
-	7650 4850 7700 4850
+	7250 4850 7700 4850
 Connection ~ 7650 4850
 Wire Wire Line
@@
 	7250 5050 7250 5150
 Wire Wire Line
-	5700 5150 7250 5150
-Wire Wire Line
-	7250 5150 8150 5150
+	5700 5150 8150 5150
 Wire Wire Line
 	5700 5150 5700 5050
@@
 	7250 6100 7250 6200
 Wire Wire Line
-	5700 6200 7250 6200
-Wire Wire Line
-	7250 6200 8200 6200
+	5700 6200 8200 6200
 Wire Wire Line
 	5700 6100 5700 6200
@@
 	7250 3950 7250 4050
 Wire Wire Line
-	5700 4050 7250 4050
-Wire Wire Line
-	7250 4050 8200 4050
+	5700 4050 8200 4050
 Wire Wire Line
 	5700 4050 5700 3950
@@
 	7250 2800 7250 2900
 Wire Wire Line
-	5700 2900 7250 2900
-Wire Wire Line
-	7250 2900 8200 2900
+	5700 2900 8200 2900
 Wire Wire Line
 	5700 2900 5700 2800
 Wire Wire Line
-	5700 2800 4800 2800
+	4800 2800 5700 2800
 Connection ~ 4800 2800
 Wire Wire Line
-	5700 3950 4800 3950
+	4800 3950 5700 3950
 Connection ~ 4800 3950
 Wire Wire Line
-	5700 5050 4800 5050
+	4800 5050 5700 5050
 Connection ~ 4800 5050
 Wire Wire Line
@@
 	8500 3300 9400 3300
 Wire Wire Line
-	4800 2100 6600 2100
-Wire Wire Line
-	6600 2100 7350 2100
-Wire Wire Line
-	7350 2100 8500 2100
+	4800 2100 8500 2100
 Wire Wire Line
 	8500 2100 8500 3300
@@
 Connection ~ 3450 5900
 Wire Wire Line
-	7250 1300 7350 1300
-Wire Wire Line
-	7350 1300 7650 1300
-Wire Wire Line
-	7650 1300 8600 1300
+	7250 1300 8600 1300
 Wire Wire Line
 	6600 1950 6600 2100
 Connection ~ 6600 2100
 Wire Wire Line
-	3450 1300 4800 1300
-Wire Wire Line
-	4800 1300 5950 1300
+	3450 1300 5950 1300
 Connection ~ 7250 2900
 Wire Wire Line
-	4800 2100 4800 2650
-Wire Wire Line
-	4800 2650 4800 2800
-Wire Wire Line
-	4800 2800 4800 3800
-Wire Wire Line
-	4800 3800 4800 3950
-Wire Wire Line
-	4800 3950 4800 4900
-Wire Wire Line
-	4800 4900 4800 5050
-Wire Wire Line
-	4800 5050 4800 5950
-Wire Wire Line
-	4800 5950 4800 6100
+	4800 2100 4800 6100
 Connection ~ 7250 4050
 Connection ~ 7250 5150
@@
 	8200 3750 8150 3750
 Wire Wire Line
-	7250 3750 7650 3750
-Wire Wire Line
-	7650 3750 7750 3750
+	7250 3750 7750 3750
 Wire Wire Line
 	8200 2900 8200 2600
@@
 	8200 2600 8150 2600
 Wire Wire Line
-	7250 2600 7650 2600
-Wire Wire Line
-	7650 2600 7750 2600
+	7250 2600 7750 2600
 Wire Wire Line
 	6700 2350 7250 2350
@@
 	7250 4600 7250 4750
 Wire Wire Line
-	7250 5900 7650 5900
-Wire Wire Line
-	7650 5900 7700 5900
+	7250 5900 7700 5900
 Wire Wire Line
 	8100 5900 8200 5900
@@
 	8200 5900 8200 6200
 Wire Wire Line
-	7650 1300 7650 2600
-Wire Wire Line
-	7650 2600 7650 3750
-Wire Wire Line
-	7650 3750 7650 4850
-Wire Wire Line
-	7650 4850 7650 5900
+	7650 1300 7650 5900
 Connection ~ 7650 5900
 Connection ~ 7650 3750
@@
 Connection ~ 7650 1300
 Wire Wire Line
-	3450 1300 3450 2600
-Wire Wire Line
-	3450 2600 3450 3750
-Wire Wire Line
-	3450 3750 3450 4850
-Wire Wire Line
-	3450 4850 3450 5900
+	3450 1300 3450 5900
 Wire Wire Line
 	6700 5650 7250 5650

Commit message: Updated schematics and documentation
Updated schematics and documentation
Parts:
- removed R3: 2000, ~, symbol R-RESCUE-Project_Narwhal_Electrical
- added R: 2000, ~, symbol R-RESCUE-Project_Narwhal_Electrical
- renumbered R4 to R, R2 to R, R3 to R
Connections:
- net GND_12V: now also R.2
- net RTD0_A: now also R.1
- net RTD0_B: now also R.1, R.1
- net at 22-23-2031.1 (P1): no longer R.1
- net at 22-23-2031.2 (PM): no longer R.1
- net at 22-23-2031.3 (P3): no longer R.1
- net at 22-23-2031.1 (P1): now also R.1; no longer R.1 (x3)
- net at 22-23-2031.2 (PM): now also R.1; no longer R.1 (x3)
- net at 22-23-2031.3 (P3): now also R.1; no longer R.1 (x3)
- net at R.2: now also R.1, R.1; no longer R.1
- new net: R.1, R.1, R.2 (x3)
Other:
- moved on the sheet: 22-23-2031, R
